File: alpakka.kicad_pcb (KiCad board)
At the start: 2 copper layers, 130 x 51 mm, 94 parts, among them P1 Debug, P2 Endpoint, P3 Conn_01x02, Q1 Q_PMOS_DGS, U1 Raspberry_Pico, U10 ST_LSM6, U12 ST_LSM6, U2 Alpsalpine_RKJXV, U3 Alpsalpine_EC10E, U4 Alpsalpine_RKJXM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

Commit message: components added, not wired
Parts:
- added C10: 100nf, ILO_fp:0402, B.Cu at (99.2, 65.8)
- added C11: 100nf, ILO_fp:0402, B.Cu at (102.1, 55.8)
- added C12: 2,2µf, ILO_fp:0402, B.Cu at (102.2, 54.2)
- added C13: 100nf, ILO_fp:0402, B.Cu at (100.0, 55.4)
- added C14: 100nf, ILO_fp:0402, B.Cu at (94.5, 59.8)
- added C15: 100nf, ILO_fp:0402, B.Cu at (94.5, 63.4)
- added C16: 100nf, ILO_fp:0402, B.Cu at (104.9, 59.2)
- added C17: 100nf, ILO_fp:0402, B.Cu at (104.9, 64.0)
- added C18: 100nf, ILO_fp:0402, B.Cu at (-7.31, 30.3)
- added C19: 2,2µf, ILO_fp:0402, B.Cu at (-7.60, 47.8)
- added C20: 100nf, ILO_fp:0402, B.Cu at (93.8, 77.8)
- added C21: 2,2µf, ILO_fp:0402, B.Cu at (93.8, 75.4)
- added C22: 1µf+, ILO_fp:0402, B.Cu at (94.0, 44.0)
- added C23: 2,2µf+, ILO_fp:0402, B.Cu at (92.4, 44.0)
- added C27: 100nf, ILO_fp:0402, B.Cu at (93.0, 49.6)
- added C8: TBD, ILO_fp:0402, B.Cu at (97.9, 49.6)
- added C9: TBD, ILO_fp:0402, B.Cu at (96.5, 54.8)
- added D5: D_Small, Diode_SMD:D_SOD-323, B.Cu at (96.8, 45.6)
- added D7: LED_GREEN, ILO_fp:0603_d, B.Cu at (93.8, 37.4)
- added D9: LED_GREEN_PWR, ILO_fp:0603_d, B.Cu at (106.2, 37.4)
- added J3: Debug, Connector_PinSocket_2.54mm:PinSocket_1x03_P2.54mm_Vertical, B.Cu at (102.4, 84.4)
- added J4: USB_C_Receptacle_USB2.0, Connector_USB:USB_C_Receptacle_G-Switch_GT-USB-7010ASV, B.Cu at (100.0, 39.2)
- added R10: 1kΩ, ILO_fp:0402, B.Cu at (98.6, 55.4)
- added R12: 1kΩ, ILO_fp:0402, B.Cu at (94.0, 70.6)
- added R13: 2kΩ, ILO_fp:0402, B.Cu at (95.4, 49.6)
- added R18: 470Ω, ILO_fp:0402, B.Cu at (106.2, 40.4)
- added R19: 5,1kΩ, ILO_fp:0402, B.Cu at (101.4, 45.6)
- added R20: 470Ω, ILO_fp:0402, B.Cu at (93.8, 41.2)
- added R22: 5,1kΩ, ILO_fp:0402, B.Cu at (98.6, 45.6)
- added R8: 27Ω, ILO_fp:0402, B.Cu at (101.2, 66.4)
- added R9: 27Ω, ILO_fp:0402, B.Cu at (102.8, 66.4)
- added RV1: Varistor, ILO_fp:0402, B.Cu at (-15.3, 35.3)
- added RV2: Varistor, ILO_fp:0402, B.Cu at (-7.30, 40.2)
- added RV3: Varistor, ILO_fp:0402, B.Cu at (102.8, 45.6)
- added SW1: SW_MEC_5G, DIY:R-668048, B.Cu at (103.3, 73.2)
- added U11: LP2985-3.3, Package_TO_SOT_SMD:SOT-23-5, B.Cu at (93.6, 47.0)
- added U5: RP2040, Package_DFN_QFN:QFN-56-1EP_7x7mm_P0.4mm_EP3.2x3.2mm, B.Cu at (100.0, 60.8)
- added U7: LM4040DBZ-3, Package_TO_SOT_SMD:SOT-23, B.Cu at (93.4, 52.4)
- added U9: W25Q16JVSSIQ, Package_SO:SOIC-8_5.23x5.23mm_P1.27mm, B.Cu at (97.6, 74.0)
- added Y1: Crystal_16Mhz, Crystal:Crystal_SMD_5032-4Pin_5.0x3.2mm, B.Cu at (98.0, 52.2)
- R1, R2, R3, R4: footprint ILO_fp:0603 -> ILO_fp:0402
- moved G*** 0.75 mm to (96.6, 80.0)
Connections:
- TP33 pad 1: GNDA -> GND
- U1 pad 33: GNDA -> GND
- U10 pad 7: GNDA -> GND
- U12 pad 7: GNDA -> GND
- U6 pad 13: GND -> /A11
Routing:
- net GNDA: track 155.4 -> 0.00 mm, vias 4 -> 0
- net GND: track 77.5 -> 229.9 mm, vias 8 -> 12
- net /A11: track 0.00 -> 3.00 mm

Commit message: finished routing
Parts:
- removed C15, C27: 100nf, ILO_fp:0402
- removed C21: 2,2µf, ILO_fp:0402
- removed R13: 2kΩ, ILO_fp:0402
- removed RV1, RV2, RV3: Varistor, ILO_fp:0402
- removed U9: W25Q16JVSSIQ, Package_SO:SOIC-8_5.23x5.23mm_P1.27mm
- SW1: footprint DIY:R-668048 -> Button_Switch_SMD:SW_Push_SPST_NO_Alps_SKRK
- U7: value LM4040DBZ-3 -> W25Q16JVUXIQ; footprint Package_TO_SOT_SMD:SOT-23 -> Package_SON:SON-8-1EP_3x2mm_P0.5mm_EP1.4x1.6mm
- Y1: footprint Crystal:Crystal_SMD_5032-4Pin_5.0x3.2mm -> Crystal:Crystal_SMD_2016-4Pin_2.0x1.6mm
- moved C18 118.7 mm to (107.5, 60.5), turned to 0 degrees
- moved C19 102.6 mm to (94.8, 54.5)
- moved D7 27.9 mm to (93.6, 65.3), turned to 90 degrees
- moved C20 24.5 mm to (104.4, 55.7), turned to 90 degrees
- moved C8 21.5 mm to (102.2, 70.7), turned to 0 degrees
- moved R20 20.3 mm to (93.6, 61.5), turned to -90 degrees
- moved Y1 16.9 mm to (102.2, 68.6), turned to 0 degrees
- moved C9 15.2 mm to (99.5, 69.7)
- moved R9 15.2 mm to (96.9, 52.4), turned to -90 degrees
- moved R8 14.3 mm to (98.5, 52.4), turned to 90 degrees
- moved R12 12.6 mm to (106.6, 70.8), turned to 0 degrees
- moved R10 11.8 mm to (102.0, 66.7), turned to 0 degrees
- moved C16 10.7 mm to (94.8, 55.9), turned to 0 degrees
- moved U7 8.40 mm to (101.8, 52.2)
- moved C12 7.48 mm to (94.8, 53.1), turned to 0 degrees
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Connections:
- U5 pad 43: VCCA -> VCC
- U7 pad 1: VCCA -> QSPI_SS
- U7 pad 2: GND -> QSPI_SD1
- U7 pad 3: (no net) -> QSPI_SD2
Routing:
- net GND: track 229.9 -> 301.5 mm, vias 12 -> 22
- net VCC: track 22.2 -> 61.8 mm, vias 5 -> 11
- net QSPI_SS: track 0.00 -> 27.3 mm, vias 0 -> 2
- net UART_TX: track 15.8 -> 40.3 mm
- net UART_RX: track 14.0 -> 36.2 mm
- net VBUS: track 11.8 -> 32.6 mm, vias 1 -> 2
- net I2C_SCL: track 121.9 -> 141.6 mm, vias 2 -> 4
- net +1V1: track 0.00 -> 19.6 mm, vias 0 -> 2
- net SPI_RX: track 142.1 -> 161.0 mm
- net GP2: track 16.3 -> 34.0 mm
- net I2C_SDA: track 124.3 -> 141.7 mm
- net SWCLK: track 0.00 -> 17.2 mm
- net GP3: track 23.1 -> 38.7 mm
- net CS0: track 71.8 -> 87.4 mm
- net SWD: track 0.00 -> 15.2 mm
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- added copper zone on B.Cu, net +1V1

Commit message: and a bit more
Routing:
- net GND: track 301.5 -> 301.0 mm
Other:
- board text added: "GND"
- board text added: "SWCLK"
- board text added: "SWD"
