File: alpakka.kicad_sch (KiCad schematic)
At the start: 76 parts, among them P1 Debug, P2 Endpoint, P3 Conn_01x02, Q1 Q_PMOS_DGS, U1 Raspberry_Pico, U10 ST_LSM6, U12 ST_LSM6, U2 Alpsalpine_RKJXV, U3 Alpsalpine_EC10E, U4 Alpsalpine_RKJXM, U6 NXP_PCAL6416A, U8 NXP_PCAL6416A

Commit message: components added, not wired
Parts:
- added C1, C2: TBD, ILO_fp:0402, symbol Device:C_Small
- added C10, C11, C12 (x2), C13, C4, C5, C7, C8, C9: 100nf, ILO_fp:0402, symbol Device:C_Small
- added C14, C15, C6: 2,2µf, ILO_fp:0402, symbol Device:C_Polarized_Small
- added C22: 1µf+, ILO_fp:0402, symbol Device:C_Small
- added C23: 2,2µf+, ILO_fp:0402, symbol Device:C_Small
- added D1: D_Small, Diode_SMD:D_SOD-323, symbol Device:D_Small
- added D2: LED_GREEN, ILO_fp:0603_d, symbol Device:LED
- added D4: LED_GREEN_PWR, ILO_fp:0603_d, symbol Device:LED
- added J10: Debug, Connector_PinSocket_2.54mm:PinSocket_1x03_P2.54mm_Vertical, symbol Connector_Generic:Conn_01x03
- added J7: USB_C_Receptacle_USB2.0, Connector_USB:USB_C_Receptacle_G-Switch_GT-USB-7010ASV, symbol Connector:USB_C_Receptacle_USB2.0
- added R1, R4: 1kΩ, ILO_fp:0402, symbol Device:R_Small
- added R10, R12: 470Ω, ILO_fp:0402, symbol Device:R_Small
- added R13, R14: 27Ω, ILO_fp:0402, symbol Device:R_Small
- added R15, R16: 5,1kΩ, ILO_fp:0402, symbol Device:R_Small
- added R5: 2kΩ, ILO_fp:0402, symbol Device:R_Small
- added RV1, RV2 (x2): Varistor, ILO_fp:0402, symbol Device:Varistor
- added SW1: SW_MEC_5G, DIY:R-668048, symbol Switch:SW_MEC_5G
- added U1: RP2040, Package_DFN_QFN:QFN-56-1EP_7x7mm_P0.4mm_EP3.2x3.2mm, symbol MCU_RaspberryPi:RP2040
- added U11: LP2985-3.3, Package_TO_SOT_SMD:SOT-23-5, symbol Regulator_Linear:LP2985-3.3
- added U2: W25Q16JVSSIQ, Package_SO:SOIC-8_5.23x5.23mm_P1.27mm, symbol Memory_Flash:W25Q32JVSS
- added U3: LM4040DBZ-3, Package_TO_SOT_SMD:SOT-23, symbol Reference_Voltage:LM4040DBZ-3
- added Y1: Crystal_16Mhz, Crystal:Crystal_SMD_5032-4Pin_5.0x3.2mm, symbol Device:Crystal_GND24_Small
- R1, R2, R3, R4: footprint ILO_fp:0603 -> ILO_fp:0402
Connections:
- net GNDA is gone; now on net GND: TP33.1, U1.33 (GND), U10.7 (GND), U12.7 (GND)
- net ADC0: now also U1.38 (GPIO26_ADC0)
- net ADC1: now also U1.39 (GPIO27_ADC1)
- net CS0: now also U1.29 (GPIO18)
- net CS1: now also U1.30 (GPIO19)
- net GND: now also C1.1, C10.1, C11.2, C12.1, C12.2, C13.2, C14.2, C15.2, C2.1, C22.1, C23.2, C4.1, C5.1, C6.1, C7.1, C8.1, C9.2, D2.1 (K), D4.1 (K), J10.2 (Pin_2), J7.A1 (GND), J7.A12 (GND), J7.B1 (GND), J7.B12 (GND), J7.S1 (SHIELD), R15.2, R16.1, RV1.2, RV2.1, RV2.2, SW1.1 (A), SW1.2 (A), U1.19 (TESTEN), U1.57 (GND), U11.2 (GND), U2.4 (GND), U3.2 (A), Y1.2, Y1.4; no longer U6.13 (P11)
- net GP2: now also U1.4 (GPIO2)
- net GP20: now also U1.31 (GPIO20)
- net GP3: now also U1.5 (GPIO3)
- net GP4: now also U1.6 (GPIO4)
- net GP5: now also U1.7 (GPIO5)
- net GP6: now also U1.8 (GPIO6)
- net GP7: now also U1.9 (GPIO7)
- net GP8: now also U1.11 (GPIO8)
- net GP9: now also U1.12 (GPIO9)
- net I2C_SCL: now also U1.18 (GPIO15)
- net I2C_SDA: now also U1.17 (GPIO14)
- net RUN: now also U1.26 (RUN)
- net SPI_CK: now also U1.13 (GPIO10)
- net SPI_RX: now also U1.15 (GPIO12)
- net SPI_TX: now also U1.14 (GPIO11)
- net UART_RX: now also U1.3 (GPIO1)
- net UART_TX: now also U1.2 (GPIO0)
- net VCCA: now also C12.2, R5.2, U1.43 (ADC_AVDD), U3.1 (K)
- net VSYS: now also C22.2, D1.1 (K), U11.1 (VIN), U11.3 (ON/~{OFF})
- net VBUS renamed +5V
- net +5V: now also D1.2 (A), J7.A4 (VBUS), J7.A9 (VBUS), J7.B4 (VBUS), J7.B9 (VBUS), RV2.2
- net VCC renamed +3.3V
- net +3.3V: now also C10.2, C11.1, C12.1, C13.1, C14.1, C15.1, C23.1, C7.2, C8.2, C9.1, R12.1, R5.1, U1.1 (IOVDD), U1.10 (IOVDD), U1.22 (IOVDD), U1.33 (IOVDD), U1.42 (IOVDD), U1.44 (VREG_IN), U1.48 (USB_VDD), U1.49 (IOVDD), U11.5 (VOUT), U2.8 (VCC)
- new net: C1.2, U1.20 (XIN), Y1.3
- new net: D2.2 (A), R10.2
- new net: J7.B5 (CC2), R15.1
- new net: R4.1, SW1.3 (B), SW1.4 (B)
- new net: D4.2 (A), R12.2
- new net: C2.2, R1.2, Y1.1
- new net: R1.1, U1.21 (XOUT)
- new net: J7.A5 (CC1), R16.2
- new net +1V1: C4.2, C5.2, C6.2, U1.23 (DVDD), U1.45 (VREG_VOUT), U1.50 (DVDD)
- new net A11: U6.13 (P11)
- new net D+: J7.A6 (D+), J7.B6 (D+), R13.2, RV1.1
- new net D-: J7.A7 (D-), J7.B7 (D-), R14.1, RV2.1
- new net DN: R14.2, U1.46 (USB_DM)
- new net DP: R13.1, U1.47 (USB_DP)
- new net GP25: R10.1, U1.37 (GPIO25)
- new net QSPI_SCLK: U1.52 (QSPI_SCLK), U2.6 (CLK)
- new net QSPI_SD0: U1.53 (QSPI_SD0), U2.5 (DI(IO0))
- new net QSPI_SD1: U1.55 (QSPI_SD1), U2.2 (DO(IO1))
- new net QSPI_SD2: U1.54 (QSPI_SD2), U2.3 (IO2)
- new net QSPI_SD3: U1.51 (QSPI_SD3), U2.7 (IO3)
- new net QSPI_SS: R4.2, U1.56 (QSPI_SS), U2.1 (~{CS})
- new net SWCLK: J10.1 (Pin_1), U1.24 (SWCLK)
- new net SWD: J10.3 (Pin_3), U1.25 (SWD)
- no-connect marks 26 -> 38
Other:
- company: Input Labs Oy. -> Input Labs, Rasmus L.
- moved on the sheet: C1, C2, C3, C4, C5, C6, D1, D2, D3, D4, P1, P2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

Commit message: finished routing
Parts:
- removed C12, C9: 100nf, ILO_fp:0402, symbol Device:C_Small
- removed C15: 2,2µf, ILO_fp:0402, symbol Device:C_Polarized_Small
- removed R5: 2kΩ, ILO_fp:0402, symbol Device:R_Small
- removed RV1, RV2 (x2): Varistor, ILO_fp:0402, symbol Device:Varistor
- removed U3: LM4040DBZ-3, Package_TO_SOT_SMD:SOT-23, symbol Reference_Voltage:LM4040DBZ-3
- SW1: footprint DIY:R-668048 -> Button_Switch_SMD:SW_Push_SPST_NO_Alps_SKRK
- U2: value W25Q16JVSSIQ -> W25Q16JVUXIQ; footprint Package_SO:SOIC-8_5.23x5.23mm_P1.27mm -> Package_SON:SON-8-1EP_3x2mm_P0.5mm_EP1.4x1.6mm
- Y1: footprint Crystal:Crystal_SMD_5032-4Pin_5.0x3.2mm -> Crystal:Crystal_SMD_2016-4Pin_2.0x1.6mm
Connections:
- net +3.3V: now also U1.43 (ADC_AVDD)
- net VCCA: no longer U1.43 (ADC_AVDD)
Other:
- moved on the sheet: C10, C11, C12, C13, C14

Commit message: changed crystal to a more common size
Parts:
- Y1: footprint Crystal:Crystal_SMD_2016-4Pin_2.0x1.6mm -> Crystal:Crystal_SMD_2520-4Pin_2.5x2.0mm
Changed lines of the file:
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@@
       (effects (font (size 1.27 1.27)))
     )
-    (property "Footprint" "Crystal:Crystal_SMD_2016-4Pin_2.0x1.6mm" (at 132.08 96.52 0)
+    (property "Footprint" "Crystal:Crystal_SMD_2520-4Pin_2.5x2.0mm" (at 132.08 96.52 0)
       (effects (font (size 1.27 1.27)) hide)
     )
